File: switching/switching.kicad_sch (KiCad schematic)
At the start: 6 parts, among them J1 Pico uC, Q1 STD60N3LH5

Commit message: circuit
Parts:
- removed J1: Pico uC, symbol Connector:Conn_01x06_Pin
- added J1: RP2040 Pico uC, symbol Connector:Conn_01x07_Pin
- added J2: MAX6675, symbol Connector:Conn_01x05_Pin
- BT1: value 18V Power -> 30V Power
- R1: value Metal Plate -> Metal Plate 10 Ohm
Connections:
- net Earth: now also J1.7 (Pin_7), J2.1 (Pin_1)
- net at R2.2: now also J1.6 (Pin_6)
- new net: J1.1 (Pin_1), J2.2 (Pin_2)
- new net: J1.4 (Pin_4), J2.3 (Pin_3)
- new net: J1.3 (Pin_3), J2.4 (Pin_4)
- new net: J1.2 (Pin_2), J2.5 (Pin_5)
Other:
- note added: "CS GP17"
- note added: "PWM GP22"
- note added: "RX GP16"
- note added: "SCK GP18"
- note added: "SDI NC"
- note added: "SO"
- note added: "VBUS"
- note added: "VCC"
- note removed: "3.3v"
- note removed: "SDI"
- note removed: "SDO"
Changed lines of the file:
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@@
   (junction (at 72.39 69.85) (diameter 0) (color 0 0 0 0)
   )
+  (junction (at 100.33 44.45) (diameter 0) (color 0 0 0 0)
+  )
   (junction (at 72.39 59.69) (diameter 0) (color 0 0 0 0)
   )
-  (wire (pts (xy 55.88 69.85) (xy 72.39 69.85))
+  (wire (pts (xy 49.53 38.1) (xy 59.69 38.1))
     (stroke (width 0) (type default))
   )
@@
     (stroke (width 0) (type default))
   )
+  (wire (pts (xy 53.34 57.15) (xy 50.8 57.15))
+    (stroke (width 0) (type default))
+  )
+  (wire (pts (xy 59.69 62.23) (xy 50.8 62.23))
+    (stroke (width 0) (type default))
+  )
   (wire (pts (xy 81.28 52.07) (xy 81.28 54.61))
     (stroke (width 0) (type default))
@@
     (stroke (width 0) (type default))
   )
-  (wire (pts (xy 55.88 67.31) (xy 63.5 67.31))
-    (stroke (width 0) (type default))
-  )
   (wire (pts (xy 63.5 67.31) (xy 63.5 59.69))
     (stroke (width 0) (type default))
   )
+  (wire (pts (xy 49.53 33.02) (xy 100.33 33.02))
+    (stroke (width 0) (type default))
+  )
   (wire (pts (xy 81.28 64.77) (xy 81.28 69.85))
     (stroke (width 0) (type default))
   )
+  (wire (pts (xy 49.53 43.18) (xy 53.34 43.18))
+    (stroke (width 0) (type default))
+  )
+  (wire (pts (xy 100.33 33.02) (xy 100.33 44.45))
+    (stroke (width 0) (type default))
+  )
+  (wire (pts (xy 50.8 67.31) (xy 63.5 67.31))
+    (stroke (width 0) (type default))
+  )
+  (wire (pts (xy 55.88 59.69) (xy 50.8 59.69))
+    (stroke (width 0) (type default))
+  )
   (wire (pts (xy 81.28 69.85) (xy 100.33 69.85))
     (stroke (width 0) (type default))
   )
+  (wire (pts (xy 53.34 43.18) (xy 53.34 57.15))
+    (stroke (width 0) (type default))
+  )
   (wire (pts (xy 71.12 59.69) (xy 72.39 59.69))
     (stroke (width 0) (type default))
   )
+  (wire (pts (xy 43.18 54.61) (xy 50.8 54.61))
+    (stroke (width 0) (type default))
+  )
+  (wire (pts (xy 59.69 38.1) (xy 59.69 62.23))
+    (stroke (width 0) (type default))
+  )
+  (wire (pts (xy 49.53 40.64) (xy 55.88 40.64))
+    (stroke (width 0) (type default))
+  )
   (wire (pts (xy 90.17 44.45) (xy 81.28 44.45))
     (stroke (width 0) (type default))
@@
     (stroke (width 0) (type default))
   )
+  (wire (pts (xy 43.18 35.56) (xy 43.18 54.61))
+    (stroke (width 0) (type default))
+  )
+  (wire (pts (xy 50.8 69.85) (xy 72.39 69.85))
+    (stroke (width 0) (type default))
+  )
+  (wire (pts (xy 49.53 35.56) (xy 43.18 35.56))
+    (stroke (width 0) (type default))
+  )
   (wire (pts (xy 100.33 44.45) (xy 100.33 69.85))
     (stroke (width 0) (type default))
@@
     (stroke (width 0) (type default))
   )
-  (text "SDO\n" (at 45.72 59.69 0)
-    (effects (font (size 1.27 1.27)) (justify left bottom))
-  )
-  (text "3.3v" (at 45.72 67.31 0)
-    (effects (font (size 1.27 1.27)) (justify left bottom))
-  )
-  (text "SDI\n" (at 45.72 62.23 0)
+  (wire (pts (xy 55.88 40.64) (xy 55.88 59.69))
+    (stroke (width 0) (type default))
+  )
+  (text "CS" (at 39.37 40.64 0)
+    (effects (font (size 1.27 1.27)) (justify left bottom))
+  )
+  (text "VBUS" (at 34.29 54.61 0)
+    (effects (font (size 1.27 1.27)) (justify left bottom))
+  )
+  (text "SO" (at 39.37 43.18 0)
     (effects (font (size 1.27 1.27)) (justify left bottom))
   )
@@
     (effects (font (size 1.27 1.27)) (justify left bottom))
   )
-  (text "GND" (at 45.72 69.85 0)
-    (effects (font (size 1.27 1.27)) (justify left bottom))
-  )
-  (text "SCK" (at 45.72 64.77 0)
-    (effects (font (size 1.27 1.27)) (justify left bottom))
-  )
-  (text "CS\n\n" (at 57.15 59.69 0)
+  (text "PWM GP22" (at 34.29 67.31 0)
+    (effects (font (size 1.27 1.27)) (justify left bottom))
+  )
+  (text "GND" (at 39.37 33.02 0)
+    (effects (font (size 1.27 1.27)) (justify left bottom))
+  )
+  (text "SDI NC" (at 34.29 64.77 0)
+    (effects (font (size 1.27 1.27)) (justify left bottom))
+  )
+  (text "CS GP17" (at 34.29 59.69 0)
+    (effects (font (size 1.27 1.27)) (justify left bottom))
+  )
+  (text "VCC" (at 39.37 35.56 0)
+    (effects (font (size 1.27 1.27)) (justify left bottom))
+  )
+  (text "RX GP16" (at 34.29 57.15 0)
+    (effects (font (size 1.27 1.27)) (justify left bottom))
+  )
+  (text "SCK GP18\n" (at 34.29 62.23 0)
+    (effects (font (size 1.27 1.27)) (justify left bottom))
+  )
+  (text "GND" (at 40.64 69.85 0)
+    (effects (font (size 1.27 1.27)) (justify left bottom))
+  )
+  (text "SCK" (at 39.37 38.1 0)
     (effects (font (size 1.27 1.27)) (justify left bottom))
   )
@@
     )
   )
+  (symbol (lib_id "Connector:Conn_01x05_Pin") (at 44.45 38.1 0) (unit 1)
+    (in_bom yes) (on_board yes) (dnp no)
+    (property "Reference" "J2" (at 45.085 29.21 0)
+      (effects (font (size 1.27 1.27)))
+    )
+    (property "Value" "MAX6675" (at 52.07 29.21 0)
+      (effects (font (size 1.27 1.27)))
+    )
+    (property "Footprint" "" (at 44.45 38.1 0)
+      (effects (font (size 1.27 1.27)) hide)
+    )
+    (property "Datasheet" "~" (at 44.45 38.1 0)
+      (effects (font (size 1.27 1.27)) hide)
+    )
+    (pin "1")
+    (pin "2")
+    (pin "3")
+    (pin "4")
+    (pin "5")
+    (instances
+      (project "switching"
+        (path "/5c1aab01-b68a-4fbd-84d9-a1df1ee3b38b"
+          (reference "J2") (unit 1)
+        )
+      )
+    )
+  )
   (symbol (lib_id "Device:Heater") (at 81.28 48.26 0) (unit 1)
     (in_bom yes) (on_board yes) (dnp no) (fields_autoplaced)
@@
       (effects (font (size 1.27 1.27)) (justify left))
     )
-    (property "Value" "Metal Plate" (at 83.82 50.165 0)
+    (property "Value" "Metal Plate 10 Ohm" (at 83.82 50.165 0)
       (effects (font (size 1.27 1.27)) (justify left))
     )
@@
     )
   )
-  (symbol (lib_id "Simulation_SPICE:NMOS") (at 78.74 59.69 0) (unit 1)
-    (in_bom yes) (on_board yes) (dnp no) (fields_autoplaced)
-    (property "Reference" "Q1" (at 85.09 59.055 0)
-      (effects (font (size 1.27 1.27)) (justify left))
-    )
-    (property "Value" "STD60N3LH5" (at 85.09 61.595 0)
-      (effects (font (size 1.27 1.27)) (justify left))
-    )
-    (property "Footprint" "" (at 83.82 57.15 0)
-      (effects (font (size 1.27 1.27)) hide)
-    )
-    (property "Datasheet" "https://ngspice.sourceforge.io/docs/ngspice-manual.pdf" (at 78.74 72.39 0)
-      (effects (font (size 1.27 1.27)) hide)
-    )
-    (property "Sim.Device" "NMOS" (at 78.74 76.835 0)
-      (effects (font (size 1.27 1.27)) hide)
-    )
-    (property "Sim.Type" "VDMOS" (at 78.74 78.74 0)
-      (effects (font (size 1.27 1.27)) hide)
-    )
-    (property "Sim.Pins" "1=D 2=G 3=S" (at 78.74 74.93 0)
-      (effects (font (size 1.27 1.27)) hide)
-    )
-    (pin "1")
-    (pin "2")
-    (pin "3")
-    (instances
-      (project "switching"
-        (path "/5c1aab01-b68a-4fbd-84d9-a1df1ee3b38b"
-          (reference "Q1") (unit 1)
-        )
-      )
-    )
-  )
-  (symbol (lib_id "Connector:Conn_01x06_Pin") (at 50.8 62.23 0) (unit 1)
-    (in_bom yes) (on_board yes) (dnp no) (fields_autoplaced)
-    (property "Reference" "J1" (at 51.435 53.34 0)
-      (effects (font (size 1.27 1.27)))
-    )
-    (property "Value" "Pico uC" (at 51.435 55.88 0)
-      (effects (font (size 1.27 1.27)))
-    )
-    (property "Footprint" "" (at 50.8 62.23 0)
-      (effects (font (size 1.27 1.27)) hide)
-    )
-    (property "Datasheet" "~" (at 50.8 62.23 0)
+  (symbol (lib_id "Connector:Conn_01x07_Pin") (at 45.72 62.23 0) (unit 1)
+    (in_bom yes) (on_board yes) (dnp no)
+    (property "Reference" "J1" (at 46.99 73.66 0)
+      (effects (font (size 1.27 1.27)))
+    )
+    (property "Value" "RP2040 Pico uC" (at 58.42 73.66 0)
+      (effects (font (size 1.27 1.27)))
+    )
+    (property "Footprint" "" (at 45.72 62.23 0)
+      (effects (font (size 1.27 1.27)) hide)
+    )
+    (property "Datasheet" "~" (at 45.72 62.23 0)
       (effects (font (size 1.27 1.27)) hide)
     )
@@
     (pin "5")
     (pin "6")
+    (pin "7")
     (instances
       (project "switching"
@@
     )
   )
+  (symbol (lib_id "Simulation_SPICE:NMOS") (at 78.74 59.69 0) (unit 1)
+    (in_bom yes) (on_board yes) (dnp no) (fields_autoplaced)
+    (property "Reference" "Q1" (at 85.09 59.055 0)
+      (effects (font (size 1.27 1.27)) (justify left))
+    )
+    (property "Value" "STD60N3LH5" (at 85.09 61.595 0)
+      (effects (font (size 1.27 1.27)) (justify left))
+    )
+    (property "Footprint" "" (at 83.82 57.15 0)
+      (effects (font (size 1.27 1.27)) hide)
+    )
+    (property "Datasheet" "https://ngspice.sourceforge.io/docs/ngspice-manual.pdf" (at 78.74 72.39 0)
+      (effects (font (size 1.27 1.27)) hide)
+    )
+    (property "Sim.Device" "NMOS" (at 78.74 76.835 0)
+      (effects (font (size 1.27 1.27)) hide)
+    )
+    (property "Sim.Type" "VDMOS" (at 78.74 78.74 0)
+      (effects (font (size 1.27 1.27)) hide)
+    )
+    (property "Sim.Pins" "1=D 2=G 3=S" (at 78.74 74.93 0)
+      (effects (font (size 1.27 1.27)) hide)
+    )
+    (pin "1")
+    (pin "2")
+    (pin "3")
+    (instances
+      (project "switching"
+        (path "/5c1aab01-b68a-4fbd-84d9-a1df1ee3b38b"
+          (reference "Q1") (unit 1)
+        )
+      )
+    )
+  )
   (symbol (lib_id "Device:Battery") (at 95.25 44.45 90) (unit 1)
     (in_bom yes) (on_board yes) (dnp no) (fields_autoplaced)
@@
       (effects (font (size 1.27 1.27)))
     )
-    (property "Value" "18V Power" (at 94.869 40.64 90)
-      (effects (font (size 1.27 1.27)))
-    )
+    (property "Value" "30V Power" (at 94.869 40.64 90)
+      (effects (font (size 1.27 1.27)))
+    )
